Commit message: Added IMU method to assist in map building

File: urdf/patrol_robot.xacro (robot description, xacro)
@@ -122,4 +122,18 @@
 		<origin xyz="0 0 0.1" rpy="0 0 0"/>
 	</joint>
+<<<<<<< HEAD
+=======
+	<link name="imu_link">
+		<inertial>
+			<mass value="0.01"/>
+			<inertia ixx="1e-5" ixy="0" ixz="0" iyy="1e-5" iyz="0" izz="1e-5"/>
+		</inertial>
+	</link>
+	<joint name="imu_joint" type="fixed">
+		<parent link="chassis"/>
+		<child link="imu_link"/>
+		<origin xyz="0 0 0.05" rpy="0 0 0"/>
+	</joint>
+>>>>>>> ea4e212 (Added IMU method to assist in map building)
 <!--==========================================-->
 <!-- Gazebo 控制與物理 -->
@@ -172,13 +186,24 @@
 			<!-- 是否發布TF與里程計資料 -->
 			<publish_odom>true</publish_odom>
+<<<<<<< HEAD
 			<publish_odom_tf>true</publish_odom_tf>
 			<publish_wheel_tf>true</publish_wheel_tf>
 			<!-- 更新頻率 -->
 			<update_rate>20</update_rate>
+=======
+			<publish_odom_tf>false</publish_odom_tf>
+			<publish_wheel_tf>false</publish_wheel_tf>
+			<!-- 更新頻率 -->
+			<update_rate>30</update_rate>
+>>>>>>> ea4e212 (Added IMU method to assist in map building)
 		</plugin>
 		<!-- 將數據發佈到topic -->
 		<plugin filename="gz-sim-joint-state-publisher-system" name="gz::sim::systems::JointStatePublisher">
 			<topic>joint_states</topic>
+<<<<<<< HEAD
 			<update_rate>20</update_rate>
+=======
+			<update_rate>30</update_rate>
+>>>>>>> ea4e212 (Added IMU method to assist in map building)
 		</plugin>
 	</gazebo>
@@ -209,3 +234,31 @@
         </sensor>
     </gazebo>
+<<<<<<< HEAD
+=======
+	<gazebo>
+  		<plugin filename="gz-sim-imu-system" name="gz::sim::systems::Imu">
+		</plugin>
+	</gazebo>
+	<gazebo reference="imu_link">
+		<sensor name="mpu6050_imu" type="imu">
+			<always_on>true</always_on>
+			<update_rate>100</update_rate>
+			<visualize>true</visualize>
+			<topic>imu/data</topic>
+			<gz_frame_id>imu_link</gz_frame_id>
+			<imu>
+				<angular_velocity>
+					<x><noise type="gaussian"><mean>0.0</mean><stddev>2e-4</stddev></noise></x>
+					<y><noise type="gaussian"><mean>0.0</mean><stddev>2e-4</stddev></noise></y>
+					<z><noise type="gaussian"><mean>0.0</mean><stddev>2e-4</stddev></noise></z>
+				</angular_velocity>
+				<linear_acceleration>
+					<x><noise type="gaussian"><mean>0.0</mean><stddev>1.7e-2</stddev></noise></x>
+					<y><noise type="gaussian"><mean>0.0</mean><stddev>1.7e-2</stddev></noise></y>
+					<z><noise type="gaussian"><mean>0.0</mean><stddev>1.7e-2</stddev></noise></z>
+				</linear_acceleration>
+			</imu>
+		</sensor>
+	</gazebo>
+>>>>>>> ea4e212 (Added IMU method to assist in map building)
 </robot>

File: worlds/world.xacro (robot description, xacro)
@@ -124,5 +124,9 @@
 	<xacro:wall_func wall_name="scene12" x="5.5" y="-7" yaw="0" length="3"/>
 	<xacro:wall_func wall_name="scene13" x="7" y="-6" yaw="1.57" length="2"/>
+<<<<<<< HEAD
 	<xacro:wall_func wall_name="scene14" x="-7" y="2" yaw="1.57" length="4"/>
+=======
+	<xacro:wall_func wall_name="scene14" x="7" y="2" yaw="1.57" length="4"/>
+>>>>>>> ea4e212 (Added IMU method to assist in map building)
 	<xacro:wall_func wall_name="scene15" x="8.5" y="0" yaw="0" length="3"/>
 </world>

Commit message: Experimental automatic navigation

File: urdf/patrol_robot.xacro (robot description, xacro)
@@ -61,4 +61,5 @@
 		</inertial>
 	</link>
+	<link name="base_footprint"/>
 	<!-- 車子底盤 -->
 	<link name="chassis">
@@ -92,4 +93,9 @@
 		</inertial>
 	</link>
+	<joint name="base_footprint_joint" type="fixed">
+		<parent link="base_footprint"/>
+		<child link="base_link"/>
+		<origin xyz="0 0 0" rpy="0 0 0"/>
+	</joint>
 	<!-- 將車子外觀建立在基準點上 -->
 	<joint name="base_joint" type="fixed">
